Commit message: Change model of robotic arm

File: sitl_config/robotic_arm/le_arm/urdf/le_arm.urdf.xacro (robot description, xacro)
@@ -13,30 +13,37 @@
             <inertial>
             <origin
-                xyz="0.034411 3.2244E-06 0.02029"
-                rpy="0 0 0" />
-            <mass value="0.00001" />
-            <inertia ixx="0.001" ixy="0.0" ixz="0.0" iyy="0.001" iyz="0.0" izz="0.001" />
-            </inertial>
-            <visual>
-            <origin
-                xyz="0 0 0"
-                rpy="0 0 0" />
-            <geometry>
-                <mesh
-                filename="package://le_arm/meshes/arm/base_link.STL" />
-            </geometry>
-            <material
-                name="">
-                <color
-                rgba="0.75294 0.75294 0.75294 1" />
-            </material>
-            </visual>
-            <collision>
-            <origin
-                xyz="0 0 0"
-                rpy="0 0 0" />
-            <geometry>
-                <mesh
-                filename="package://le_arm/meshes/arm/base_link.STL" />
+                xyz="6.8888E-08 0.0005198 -0.060933"
+                rpy="0 0 0" />
+            <mass
+                value="0.23834" />
+            <inertia
+                ixx="0.00014646"
+                ixy="-4.6203E-05"
+                ixz="2.9588E-12"
+                iyy="0.00021227"
+                iyz="-5.2784E-06"
+                izz="0.00027887" />
+            </inertial>
+            <visual>
+            <origin
+                xyz="0 0 0"
+                rpy="0 0 0" />
+            <geometry>
+                <mesh
+                filename="package://le_arm/meshes/arm_base_link.STL" />
+            </geometry>
+            <material
+                name="">
+                <color
+                rgba="0.64706 0.51765 0 1" />
+            </material>
+            </visual>
+            <collision>
+            <origin
+                xyz="0 0 0"
+                rpy="0 0 0" />
+            <geometry>
+                <mesh
+                filename="package://le_arm/meshes/arm_base_link.STL" />
             </geometry>
             </collision>
@@ -53,30 +60,37 @@
             <inertial>
             <origin
-                xyz="-0.0005946 -0.00090913 0.017195"
-                rpy="0 0 0" />
-            <mass value="0.00001" />
-            <inertia ixx="0.001" ixy="0.0" ixz="0.0" iyy="0.001" iyz="0.0" izz="0.001" />
-            </inertial>
-            <visual>
-            <origin
-                xyz="0 0 0"
-                rpy="0 0 0" />
-            <geometry>
-                <mesh
-                filename="package://le_arm/meshes/arm/shoulder_link.STL" />
-            </geometry>
-            <material
-                name="">
-                <color
-                rgba="0.75294 0.75294 0.75294 1" />
-            </material>
-            </visual>
-            <collision>
-            <origin
-                xyz="0 0 0"
-                rpy="0 0 0" />
-            <geometry>
-                <mesh
-                filename="package://le_arm/meshes/arm/shoulder_link.STL" />
+                xyz="-0.0071984 5.2965E-07 -0.040115"
+                rpy="0 0 0" />
+            <mass
+                value="0.087666" />
+            <inertia
+                ixx="3.1627E-05"
+                ixy="-3.6677E-10"
+                ixz="5.4309E-06"
+                iyy="3.0921E-05"
+                iyz="-2.1161E-09"
+                izz="3.7509E-05" />
+            </inertial>
+            <visual>
+            <origin
+                xyz="0 0 0"
+                rpy="0 0 0" />
+            <geometry>
+                <mesh
+                filename="package://le_arm/meshes/shoulder_link.STL" />
+            </geometry>
+            <material
+                name="">
+                <color
+                rgba="0.89804 0.91765 0.92941 1" />
+            </material>
+            </visual>
+            <collision>
+            <origin
+                xyz="0 0 0"
+                rpy="0 0 0" />
+            <geometry>
+                <mesh
+                filename="package://le_arm/meshes/shoulder_link.STL" />
             </geometry>
             </collision>
@@ -93,6 +107,6 @@
             type="revolute">
             <origin
-            xyz="0.0005 0 0.0535"
-            rpy="1.2297E-10 2.2825E-27 -3.4694E-17" />
+            xyz="0 0.0895 0"
+            rpy="2.4302 1.5708 0" />
             <parent
             link="arm_base_link" />
@@ -100,10 +114,10 @@
             link="shoulder_link" />
             <axis
-            xyz="0 0 1" />
+            xyz="-1 0 0" />
             <limit
-            lower="-1.57"
-            upper="1.57"
-            effort="1000"
-            velocity="2" />
+            lower="-3.14"
+            upper="3.14"
+            effort="100"
+            velocity="100" />
         </joint>
         <link
@@ -111,30 +125,37 @@
             <inertial>
             <origin
-                xyz="2.6345E-08 -0.02405 0.05197"
-                rpy="0 0 0" />
-            <mass value="0.00001" />
-            <inertia ixx="0.001" ixy="0.0" ixz="0.0" iyy="0.001" iyz="0.0" izz="0.001" />
-            </inertial>
-            <visual>
-            <origin
-                xyz="0 0 0"
-                rpy="0 0 0" />
-            <geometry>
-                <mesh
-                filename="package://le_arm/meshes/arm/upper_arm_link.STL" />
-            </geometry>
-            <material
-                name="">
-                <color
-                rgba="0.75294 0.75294 0.75294 1" />
-            </material>
-            </visual>
-            <collision>
-            <origin
-                xyz="0 0 0"
-                rpy="0 0 0" />
-            <geometry>
-                <mesh
-                filename="package://le_arm/meshes/arm/upper_arm_link.STL" />
+                xyz="-0.00072842 -0.00022202 0.02553"
+                rpy="0 0 0" />
+            <mass
+                value="0.10559" />
+            <inertia
+                ixx="0.00010233"
+                ixy="-5.0947E-08"
+                ixz="-6.5487E-07"
+                iyy="9.0284E-05"
+                iyz="-8.153E-08"
+                izz="1.8127E-05" />
+            </inertial>
+            <visual>
+            <origin
+                xyz="0 0 0"
+                rpy="0 0 0" />
+            <geometry>
+                <mesh
+                filename="package://le_arm/meshes/upper_arm_link.STL" />
+            </geometry>
+            <material
+                name="">
+                <color
+                rgba="0.89804 0.91765 0.92941 1" />
+            </material>
+            </visual>
+            <collision>
+            <origin
+                xyz="0 0 0"
+                rpy="0 0 0" />
+            <geometry>
+                <mesh
+                filename="package://le_arm/meshes/upper_arm_link.STL" />
             </geometry>
             </collision>
@@ -151,6 +172,6 @@
             type="revolute">
             <origin
-            xyz="-0.0105 0.0226 0.032"
-            rpy="-5.7183E-11 0.785 0" />
+            xyz="0 0 -0.14296"
+            rpy="3.1416 0 3.1359" />
             <parent
             link="shoulder_link" />
@@ -158,10 +179,10 @@
             link="upper_arm_link" />
             <axis
-            xyz="0 -1 0" />
+            xyz="0 0 1" />
             <limit
-            lower="-1.57"
-            upper="1.57"
-            effort="1000"
-            velocity="2" />
+            lower="-3.14"
+            upper="3.14"
+            effort="100"
+            velocity="100" />
         </joint>
         <link
@@ -169,30 +190,37 @@
             <inertial>
             <origin
-                xyz="3.5006E-08 0.0090395 0.033861"
-                rpy="0 0 0" />
-            <mass value="0.00001" />
-            <inertia ixx="0.001" ixy="0.0" ixz="0.0" iyy="0.001" iyz="0.0" izz="0.001" />
-            </inertial>
-            <visual>
-            <origin
-                xyz="0 0 0"
-                rpy="0 0 0" />
-            <geometry>
-                <mesh
-                filename="package://le_arm/meshes/arm/forearm_link.STL" />
-            </geometry>
-            <material
-                name="">
-                <color
-                rgba="0.75294 0.75294 0.75294 1" />
-            </material>
-            </visual>
-            <collision>
-            <origin
-                xyz="0 0 0"
-                rpy="0 0 0" />
-            <geometry>
-                <mesh
-                filename="package://le_arm/meshes/arm/forearm_link.STL" />
+                xyz="-0.0074811 -0.0001625 -0.039025"
+                rpy="0 0 0" />
+            <mass
+                value="0.086986" />
+            <inertia
+                ixx="3.031E-05"
+                ixy="3.5519E-10"
+                ixz="5.3565E-06"
+                iyy="3.0859E-05"
+                iyz="-1.6295E-08"
+                izz="3.7684E-05" />
+            </inertial>
+            <visual>
+            <origin
+                xyz="0 0 0"
+                rpy="0 0 0" />
+            <geometry>
+                <mesh
+                filename="package://le_arm/meshes/forearm_link.STL" />
+            </geometry>
+            <material
+                name="">
+                <color
+                rgba="0.89804 0.91765 0.92941 1" />
+            </material>
+            </visual>
+            <collision>
+            <origin
+                xyz="0 0 0"
+                rpy="0 0 0" />
+            <geometry>
+                <mesh
+                filename="package://le_arm/meshes/forearm_link.STL" />
             </geometry>
             </collision>
@@ -209,6 +237,6 @@
             type="revolute">
             <origin
-            xyz="0 -0.0335 0.104"
-            rpy="-1.6E-10 0.785 0" />
+            xyz="0 0 0.069036"
+            rpy="2.6943 0 0" />
             <parent
             link="upper_arm_link" />
@@ -216,10 +244,10 @@
             link="forearm_link" />
             <axis
-            xyz="0 -1 0" />
+            xyz="-1 0 0" />
             <limit
-            lower="-1.57"
-            upper="1.57"
-            effort="1000"
-            velocity="2" />
+            lower="-3.14"
+            upper="3.14"
+            effort="100"
+            velocity="100" />
         </joint>
         <link
@@ -227,30 +255,37 @@
             <inertial>
             <origin
-                xyz="-0.010432 0.010212 0.019017"
-                rpy="0 0 0" />
-            <mass value="0.00001" />
-            <inertia ixx="0.001" ixy="0.0" ixz="0.0" iyy="0.001" iyz="0.0" izz="0.001" />
-            </inertial>
-            <visual>
-            <origin
-                xyz="0 0 0"
-                rpy="0 0 0" />
-            <geometry>
-                <mesh
-                filename="package://le_arm/meshes/arm/wrist_1_link.STL" />
-            </geometry>
-            <material
-                name="">
-                <color
-                rgba="0.75294 0.75294 0.75294 1" />
-            </material>
-            </visual>
-            <collision>
-            <origin
-                xyz="0 0 0"
-                rpy="0 0 0" />
-            <geometry>
-                <mesh
-                filename="package://le_arm/meshes/arm/wrist_1_link.STL" />
+                xyz="0.00020523 -0.0029296 0.0079122"
+                rpy="0 0 0" />
+            <mass
+                value="0.013253" />
+            <inertia
+                ixx="2.333E-06"
+                ixy="-7.9684E-09"
+                ixz="4.9095E-09"
+                iyy="1.7076E-06"
+                iyz="1.1168E-07"
+                izz="3.0343E-06" />
+            </inertial>
+            <visual>
+            <origin
+                xyz="0 0 0"
+                rpy="0 0 0" />
+            <geometry>
+                <mesh
+                filename="package://le_arm/meshes/wrist_1_link.STL" />
+            </geometry>
+            <material
+                name="">
+                <color
+                rgba="1 1 1 1" />
+            </material>
+            </visual>
+            <collision>
+            <origin
+                xyz="0 0 0"
+                rpy="0 0 0" />
+            <geometry>
+                <mesh
+                filename="package://le_arm/meshes/wrist_1_link.STL" />
             </geometry>
             </collision>
@@ -267,6 +302,6 @@
             type="revolute">
             <origin
-            xyz="-0.0007415 0.0054 0.088419"
-            rpy="5.3884E-11 0 0" />
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