Commit message: fix bugs

File: sitl_config/models/rotors_description/urdf/iris_arm_base.xacro (robot description, xacro)
@@ -63,5 +63,5 @@
   <xacro:include filename="$(find le_arm)/urdf/le_arm.urdf.xacro" />
   <xacro:le_arm parent="base_link" >
-    <origin xyz="-0.1 0 -0.05" rpy="0 3.14 3.14"/>
+    <origin xyz="0 0 0" rpy="-1.5708 0 3.14159"/>
   </xacro:le_arm>
   <xacro:if value="$(arg enable_wind)">

File: sitl_config/robotic_arm/le_arm/urdf/le_arm.urdf.xacro (robot description, xacro)
@@ -31,5 +31,5 @@
             <geometry>
                 <mesh
-                filename="package://le_arm/meshes/arm_base_link.STL" />
+                filename="package://le_arm/meshes/arm/base_link.STL" />
             </geometry>
             <material
@@ -45,5 +45,5 @@
             <geometry>
                 <mesh
-                filename="package://le_arm/meshes/arm_base_link.STL" />
+                filename="package://le_arm/meshes/arm/base_link.STL" />
             </geometry>
             </collision>
@@ -78,5 +78,5 @@
             <geometry>
                 <mesh
-                filename="package://le_arm/meshes/shoulder_link.STL" />
+                filename="package://le_arm/meshes/arm/shoulder_link.STL" />
             </geometry>
             <material
@@ -92,5 +92,5 @@
             <geometry>
                 <mesh
-                filename="package://le_arm/meshes/shoulder_link.STL" />
+                filename="package://le_arm/meshes/arm/shoulder_link.STL" />
             </geometry>
             </collision>
@@ -143,5 +143,5 @@
             <geometry>
                 <mesh
-                filename="package://le_arm/meshes/upper_arm_link.STL" />
+                filename="package://le_arm/meshes/arm/upper_arm_link.STL" />
             </geometry>
             <material
@@ -157,5 +157,5 @@
             <geometry>
                 <mesh
-                filename="package://le_arm/meshes/upper_arm_link.STL" />
+                filename="package://le_arm/meshes/arm/upper_arm_link.STL" />
             </geometry>
             </collision>
@@ -208,5 +208,5 @@
             <geometry>
                 <mesh
-                filename="package://le_arm/meshes/forearm_link.STL" />
+                filename="package://le_arm/meshes/arm/forearm_link.STL" />
             </geometry>
             <material
@@ -222,5 +222,5 @@
             <geometry>
                 <mesh
-                filename="package://le_arm/meshes/forearm_link.STL" />
+                filename="package://le_arm/meshes/arm/forearm_link.STL" />
             </geometry>
             </collision>
@@ -273,5 +273,5 @@
             <geometry>
                 <mesh
-                filename="package://le_arm/meshes/wrist_1_link.STL" />
+                filename="package://le_arm/meshes/arm/wrist_1_link.STL" />
             </geometry>
             <material
@@ -287,5 +287,5 @@
             <geometry>
                 <mesh
-                filename="package://le_arm/meshes/wrist_1_link.STL" />
+                filename="package://le_arm/meshes/arm/wrist_1_link.STL" />
             </geometry>
             </collision>
